Commit message: Updated URDF and other improvements for the challenge

File: iiwa_stack/iiwa_description/urdf/iiwa14.urdf.xacro (robot description, xacro)
@@ -7,4 +7,5 @@
   <!--Import base GP -->
   <xacro:include filename="$(find iiwa_description)/urdf/rosie2base.xacro"/>
+  <xacro:include filename="$(find robotiq_2f_85_gripper_visualization)/urdf/robotiq_arg2f_85_model.xacro"/>
   <xacro:arg name="hardware_interface" default="PositionJointInterface"/>
   <xacro:arg name="robot_name" default="iiwa"/>

File: iiwa_stack/iiwa_description/urdf/iiwa7.urdf.xacro (robot description, xacro)
@@ -19,352 +19,3 @@
     <origin xyz="$(arg origin_xyz)" rpy="$(arg origin_rpy)" />
   </xacro:iiwa7>
-  <!-- Joint to connect to the iiwa arm -->
-  <!-- <joint name="arm_to_gripper" type="fixed">
-      <origin xyz="0 0 0" rpy="0 0 1.5708" />
-      <parent link="${robot_name}_link_ee" />
-      <child link="robotiq_arg2f_base_link" />
-      <axis xyz="0 0 0" />
-  </joint> -->
-  <!-- Frame coincident with all-zeros TCP on UR controller -->
-  <!-- <link name="$(arg robot_name)_link_ee"/> -->
-  <!-- <link name="world"/> -->
-  <!-- <joint name="world_joint" type="fixed">
-    <parent link="world"/>
-    <child link="base_link"/>
-    <origin rpy="0.0 0.0 0.0" xyz="0.0 0.0 0.0"/>
-  </joint> -->
-  <!-- Robotiq Coupler -->
-  <!--  + Height added by the coupler: 8mm -->
-  <!--  + Reference frame: at the middle (4mm) -->
-  <link name="robotiq_coupler">
-    <visual>
-      <geometry>
-        <mesh filename="package://robotiq_description/meshes/visual/robotiq_85_coupler.stl"/>
-      </geometry>
-      <material name="flat_black"/>
-    </visual>
-    <collision>
-      <geometry>
-        <mesh filename="package://robotiq_description/meshes/visual/robotiq_85_coupler.stl"/>
-      </geometry>
-    </collision>
-    <inertial>
-      <origin rpy="0 0 0" xyz="2.073e-05   1.45286e-03  -1.1049e-03"/>
-      <mass value="0.168"/>
-      <inertia ixx="6.69695624e-05" ixy="5.21511788e-09" ixz="-2.74383009e-08" iyy="7.85088161e-05" iyz="5.41105193e-07" izz="1.41819717e-04"/>
-    </inertial>
-  </link>
-  <joint name="robotiq_coupler_joint" type="fixed">
-    <origin rpy="0 0 -1.5707963267948966" xyz="0 0 0.004"/>
-    <parent link="$(arg robot_name)_link_ee"/>
-    <child link="robotiq_coupler"/>
-  </joint>
-  <gazebo reference="robotiq_coupler">
-    <mu1>0.9</mu1>
-    <mu2>0.9</mu2>
-    <material>Gazebo/FlatBlack</material>
-  </gazebo>
-  <!-- Equivalent to the OpenRAVE manipulator denso_robotiq_85_gripper -->
-  <!-- <link name="denso_robotiq_85_gripper" /> -->
-  <!-- <joint name="manipulator_dummy_joint" type="fixed"> -->
-  <!--   <origin xyz="0 0 0.1441" rpy="0 0 0" /> -->
-  <!--   <parent link="robotiq_coupler"/> -->
-  <!--   <child link="denso_robotiq_85_gripper"/> -->
-  <!-- </joint> -->
-  <joint name="robotiq_85_base_joint" type="fixed">
-    <parent link="robotiq_coupler"/>
-    <child link="robotiq_85_base_link"/>
-    <origin rpy="0 -1.5707963267948966 3.141592653589793" xyz="0 0 0.004"/>
-  </joint>
-  <link name="robotiq_85_base_link">
-    <visual>
-      <geometry>
-        <mesh filename="package://robotiq_description/meshes/visual/robotiq_85_base_link.dae"/>
-      </geometry>
-    </visual>
-    <collision>
-      <geometry>
-        <mesh filename="package://robotiq_description/meshes/collision/robotiq_85_base_link.stl"/>
-      </geometry>
-    </collision>
-    <inertial>
-      <mass value="0.636951"/>
-      <origin xyz="0.0 0.0 0.0"/>
-      <inertia ixx="0.000380" ixy="0.000000" ixz="0.000000" iyx="0.000000" iyy="0.001110" iyz="0.000000" izx="0.000000" izy="0.000000" izz="0.001171"/>
-    </inertial>
-  </link>
-  <joint name="robotiq_85_left_knuckle_joint" type="revolute">
-    <parent link="robotiq_85_base_link"/>
-    <child link="robotiq_85_left_knuckle_link"/>
-    <axis xyz="0 0 1"/>
-    <origin rpy="3.141592653589793 0.0 0.0" xyz="0.05490451627 0.03060114443 0.0"/>
-    <limit effort="1000" lower="0.0" upper="0.80285" velocity="0.5"/>
-  </joint>
-  <joint name="robotiq_85_right_knuckle_joint" type="continuous">
-    <parent link="robotiq_85_base_link"/>
-    <child link="robotiq_85_right_knuckle_link"/>
-    <axis xyz="0 0 1"/>
-    <origin rpy="0.0 0.0 0.0" xyz="0.05490451627 -0.03060114443 0.0"/>
-    <limit effort="1000" lower="-3.14" upper="3.14" velocity="100.0"/>
-    <mimic joint="robotiq_85_left_knuckle_joint"/>
-  </joint>
-  <link name="robotiq_85_left_knuckle_link">
-    <visual>
-      <geometry>
-        <mesh filename="package://robotiq_description/meshes/visual/robotiq_85_knuckle_link.dae"/>
-      </geometry>
-    </visual>
-    <collision>
-      <geometry>
-        <mesh filename="package://robotiq_description/meshes/collision/robotiq_85_knuckle_link.stl"/>
-      </geometry>
-    </collision>
-    <inertial>
-      <mass value="0.018491"/>
-      <origin xyz="0.0 0.0 0.0"/>
-      <inertia ixx="0.000009" ixy="-0.000001" ixz="0.000000" iyx="-0.000001" iyy="0.000001" iyz="0.000000" izx="0.000000" izy="0.000000" izz="0.000010"/>
-    </inertial>
-  </link>
-  <link name="robotiq_85_right_knuckle_link">
-    <visual>
-      <geometry>
-        <mesh filename="package://robotiq_description/meshes/visual/robotiq_85_knuckle_link.dae"/>
-      </geometry>
-    </visual>
-    <collision>
-      <geometry>
-        <mesh filename="package://robotiq_description/meshes/collision/robotiq_85_knuckle_link.stl"/>
-      </geometry>
-    </collision>
-    <inertial>
-      <mass value="0.018491"/>
-      <origin xyz="0.0 0.0 0.0"/>
-      <inertia ixx="0.000009" ixy="-0.000001" ixz="0.000000" iyx="-0.000001" iyy="0.000001" iyz="0.000000" izx="0.000000" izy="0.000000" izz="0.000010"/>
-    </inertial>
-  </link>
-  <joint name="robotiq_85_left_finger_joint" type="fixed">
-    <parent link="robotiq_85_left_knuckle_link"/>
-    <child link="robotiq_85_left_finger_link"/>
-    <origin rpy="0 0 0" xyz="-0.00408552455 -0.03148604435 0.0"/>
-  </joint>
-  <joint name="robotiq_85_right_finger_joint" type="fixed">
-    <parent link="robotiq_85_right_knuckle_link"/>
-    <child link="robotiq_85_right_finger_link"/>
-    <origin rpy="0 0 0" xyz="-0.00408552455 -0.03148604435 0.0"/>
-  </joint>
-  <link name="robotiq_85_left_finger_link">
-    <visual>
-      <geometry>
-        <mesh filename="package://robotiq_description/meshes/visual/robotiq_85_finger_link.dae"/>
-      </geometry>
-    </visual>
-    <collision>
-      <geometry>
-        <mesh filename="package://robotiq_description/meshes/collision/robotiq_85_finger_link.stl"/>
-      </geometry>
-    </collision>
-    <inertial>
-      <mass value="0.027309"/>
-      <origin xyz="0.0 0.0 0.0"/>
-      <inertia ixx="0.000003" ixy="-0.000002" ixz="0.000000" iyx="-0.000002" iyy="0.000021" iyz="0.000000" izx="0.000000" izy="0.000000" izz="0.000020"/>
-    </inertial>
-  </link>
-  <link name="robotiq_85_right_finger_link">
-    <visual>
-      <geometry>
-        <mesh filename="package://robotiq_description/meshes/visual/robotiq_85_finger_link.dae"/>
-      </geometry>
-    </visual>
-    <collision>
-      <geometry>
-        <mesh filename="package://robotiq_description/meshes/collision/robotiq_85_finger_link.stl"/>
-      </geometry>
-    </collision>
-    <inertial>
-      <mass value="0.027309"/>
-      <origin xyz="0.0 0.0 0.0"/>
-      <inertia ixx="0.000003" ixy="-0.000002" ixz="0.000000" iyx="-0.000002" iyy="0.000021" iyz="0.000000" izx="0.000000" izy="0.000000" izz="0.000020"/>
-    </inertial>
-  </link>
-  <joint name="robotiq_85_left_inner_knuckle_joint" type="continuous">
-    <parent link="robotiq_85_base_link"/>
-    <child link="robotiq_85_left_inner_knuckle_link"/>
-    <axis xyz="0 0 1"/>
-    <origin rpy="3.141592653589793 0.0 0.0" xyz="0.06142 0.0127 0"/>
-    <limit effort="0.1" lower="-3.14" upper="3.14" velocity="100.0"/>
-    <mimic joint="robotiq_85_left_knuckle_joint" offset="0"/>
-  </joint>
-  <joint name="robotiq_85_right_inner_knuckle_joint" type="continuous">
-    <parent link="robotiq_85_base_link"/>
-    <child link="robotiq_85_right_inner_knuckle_link"/>
-    <axis xyz="0 0 1"/>
-    <origin rpy="0 0 0" xyz="0.06142 -0.0127 0"/>
-    <limit effort="0.1" lower="-3.14" upper="3.14" velocity="100.0"/>
-    <mimic joint="robotiq_85_left_knuckle_joint" offset="0"/>
-  </joint>
-  <link name="robotiq_85_left_inner_knuckle_link">
-    <visual>
-      <geometry>
-        <mesh filename="package://robotiq_description/meshes/visual/robotiq_85_inner_knuckle_link.dae"/>
-      </geometry>
-    </visual>
-    <collision>
-      <geometry>
-        <mesh filename="package://robotiq_description/meshes/collision/robotiq_85_inner_knuckle_link.stl"/>
-      </geometry>
-    </collision>
-    <inertial>
-      <mass value="0.029951"/>
-      <origin xyz="0.0 0.0 0.0"/>
-      <inertia ixx="0.000039" ixy="0.000000" ixz="0.000000" iyx="0.000000" iyy="0.000005" iyz="0.000000" izx="0.000000" izy="0.000000" izz="0.000035"/>
-    </inertial>
-  </link>
-  <link name="robotiq_85_right_inner_knuckle_link">
-    <visual>
-      <geometry>
-        <mesh filename="package://robotiq_description/meshes/visual/robotiq_85_inner_knuckle_link.dae"/>
-      </geometry>
-    </visual>
-    <collision>
-      <geometry>
-        <mesh filename="package://robotiq_description/meshes/collision/robotiq_85_inner_knuckle_link.stl"/>
-      </geometry>
-    </collision>
-    <inertial>
-      <mass value="0.029951"/>
-      <origin xyz="0.0 0.0 0.0"/>
-      <inertia ixx="0.000039" ixy="0.000000" ixz="0.000000" iyx="0.000000" iyy="0.000005" iyz="0.000000" izx="0.000000" izy="0.000000" izz="0.000035"/>
-    </inertial>
-  </link>
-  <joint name="robotiq_85_left_finger_tip_joint" type="continuous">
-    <parent link="robotiq_85_left_inner_knuckle_link"/>
-    <child link="robotiq_85_left_finger_tip_link"/>
-    <axis xyz="0 0 1"/>
-    <origin rpy="0.0 0.0 0.0" xyz="0.04303959807 -0.03759940821 0.0"/>
-    <limit effort="0.1" lower="-3.14" upper="3.14" velocity="100.0"/>
-    <mimic joint="robotiq_85_left_knuckle_joint" multiplier="-1"/>
-  </joint>
-  <joint name="robotiq_85_right_finger_tip_joint" type="continuous">
-    <parent link="robotiq_85_right_inner_knuckle_link"/>
-    <child link="robotiq_85_right_finger_tip_link"/>
-    <axis xyz="0 0 1"/>
-    <origin rpy="0.0 0.0 0.0" xyz="0.04303959807 -0.03759940821  0.0"/>
-    <limit effort="0.1" lower="-3.14" upper="3.14" velocity="100.0"/>
-    <mimic joint="robotiq_85_left_knuckle_joint" multiplier="-1"/>
-  </joint>
-  <link name="robotiq_85_left_finger_tip_link">
-    <visual>
-      <geometry>
-        <mesh filename="package://robotiq_description/meshes/visual/robotiq_85_finger_tip_link.dae"/>
-      </geometry>
-    </visual>
-    <collision>
-      <geometry>
-        <mesh filename="package://robotiq_description/meshes/collision/robotiq_85_finger_tip_link.stl"/>
-      </geometry>
-    </collision>
-    <inertial>
-      <mass value="0.019555"/>
-      <origin xyz="0.0 0.0 0.0"/>
-      <inertia ixx="0.000002" ixy="0.000000" ixz="0.000000" iyx="0.000000" iyy="0.000005" iyz="0.000000" izx="0.000000" izy="0.000000" izz="0.000006"/>
-    </inertial>
-  </link>
-  <link name="robotiq_85_right_finger_tip_link">
-    <visual>
-      <geometry>
-        <mesh filename="package://robotiq_description/meshes/visual/robotiq_85_finger_tip_link.dae"/>
-      </geometry>
-    </visual>
-    <collision>
-      <geometry>
-        <mesh filename="package://robotiq_description/meshes/collision/robotiq_85_finger_tip_link.stl"/>
-      </geometry>
-    </collision>
-    <inertial>
-      <mass value="0.019555"/>
-      <origin xyz="0.0 0.0 0.0"/>
-      <inertia ixx="0.000002" ixy="0.000000" ixz="0.000000" iyx="0.000000" iyy="0.000005" iyz="0.000000" izx="0.000000" izy="0.000000" izz="0.000006"/>
-    </inertial>
-  </link>
-  <!-- Improve grasping physics -->
-  <gazebo reference="robotiq_85_left_finger_tip_link">
-    <kp>1000000.0</kp>
-    <kd>1.0</kd>
-    <mu1>1.0</mu1>
-    <mu2>1.0</mu2>
-    <minDepth>0.001</minDepth>
-  </gazebo>
-  <gazebo reference="robotiq_85_right_finger_tip_link">
-    <kp>1000000.0</kp>
-    <kd>1.0</kd>
-    <mu1>1.0</mu1>
-    <mu2>1.0</mu2>
-    <minDepth>0.001</minDepth>
-  </gazebo>
-  <transmission name="robotiq_85_left_knuckle_trans">
-    <type>transmission_interface/SimpleTransmission</type>
-    <joint name="robotiq_85_left_knuckle_joint">
-      <hardwareInterface>PositionJointInterface</hardwareInterface>
-      <!-- <hardwareInterface>hardwareInterface/EffortJointInterface</hardwareInterface> -->
-    </joint>
-    <actuator name="robotiq_85_left_knuckle_motor">
-      <mechanicalReduction>1</mechanicalReduction>
-      <hardwareInterface>PositionJointInterface</hardwareInterface>
-      <!-- <hardwareInterface>EfforJointInterface</hardwareInterface> -->
-    </actuator>
-  </transmission>
-  <!-- Mimic joints -->
-  <gazebo>
-    <plugin filename="libgazebo_mimic_joint_plugin.so" name="mimic_robotiq_85_1">
-      <joint>robotiq_85_left_knuckle_joint</joint>
-      <mimicJoint>robotiq_85_right_knuckle_joint</mimicJoint>
-    </plugin>
-    <plugin filename="libgazebo_mimic_joint_plugin.so" name="mimic_robotiq_85_2">
-      <joint>robotiq_85_left_knuckle_joint</joint>
-      <mimicJoint>robotiq_85_left_inner_knuckle_joint</mimicJoint>
-    </plugin>
-    <plugin filename="libgazebo_mimic_joint_plugin.so" name="mimic_robotiq_85_3">
-      <joint>robotiq_85_left_knuckle_joint</joint>
-      <mimicJoint>robotiq_85_right_inner_knuckle_joint</mimicJoint>
-    </plugin>
-    <plugin filename="libgazebo_mimic_joint_plugin.so" name="mimic_robotiq_85_4">
-      <joint>robotiq_85_left_knuckle_joint</joint>
-      <mimicJoint>robotiq_85_left_finger_tip_joint</mimicJoint>
-      <multiplier>-1.0</multiplier>
-      <offset>0.0</offset>
-    </plugin>
-    <plugin filename="libgazebo_mimic_joint_plugin.so" name="mimic_robotiq_85_5">
-      <joint>robotiq_85_left_knuckle_joint</joint>
-      <mimicJoint>robotiq_85_right_finger_tip_joint</mimicJoint>
-      <multiplier>-1.0</multiplier>
-      <offset>0.0</offset>
-    </plugin>
-  </gazebo>
-  <!-- Gazebo FT sensor plugin -->
-  <gazebo reference="wrist_3_joint">
-    <provideFeedback>true</provideFeedback>
-  </gazebo>
-  <gazebo>
-    <plugin filename="libgazebo_ros_ft_sensor.so" name="ft_sensor_plugin">
-      <updateRate>250.0</updateRate>
-      <topicName>ft_sensor/raw</topicName>
-      <gaussianNoise>0.0</gaussianNoise>
-      <jointName>wrist_3_joint</jointName>
-    </plugin>
-  </gazebo>
-  <!-- Gazebo grasping plugin -->
-  <gazebo>
-    <gripper name="gazebo_gripper">
-      <grasp_check>
-        <attach_steps>2</attach_steps>
-        <!-- default: 20 -->
-        <detach_steps>2</detach_steps>
-        <!-- default: 40 -->
-        <min_contact_count>3</min_contact_count>
-      </grasp_check>
-      <gripper_link>robotiq_85_left_finger_tip_link</gripper_link>
-      <gripper_link>robotiq_85_right_finger_tip_link</gripper_link>
-      <palm_link>robotiq_85_base_link</palm_link>
-    </gripper>
-  </gazebo>
 </robot>
