Commit message: Added inertia information for robotiq gripper

File: iiwa_stack/iiwa_description/urdf/iiwa_gripper.urdf (robot description, URDF)
Before this commit: robot iiwa14, 23 links, 22 joints
Links:
- link left_inner_finger: mass None -> 0.0104003125914103
- link left_inner_knuckle: mass None -> 0.0271177346495152
- link left_outer_finger: mass None -> 0.022614240507152
- link left_outer_knuckle: mass None -> 0.00853198276973456
- link right_inner_finger: mass None -> 0.0104003125914103
- link right_inner_knuckle: mass None -> 0.0271177346495152
- link right_outer_finger: mass None -> 0.022614240507152
- link right_outer_knuckle: mass None -> 0.00853198276973456
