Commit message: added plate and siegmund table to urdf

File: iiwa_stack/iiwa_description/urdf/rosie2siegmundbase.xacro (robot description, xacro)
@@ -14,15 +14,15 @@
       <inertial>
         <origin
-          xyz="-7.6417091746513E-05 0.40001338309557 0.164858799827291"
+          xyz="1 0.5 -0.13"
           rpy="0 0 0" />
         <mass
-          value="53.6277106242961" />
+          value="330" />
         <inertia
-          ixx="6.3670548916442"
-          ixy="-1.9067207201396E-05"
-          ixz="3.77494926341754E-05"
-          iyy="4.38733657045515"
-          iyz="3.54070945707606E-05"
-          izz="5.36753756395971" />
+          ixx="139.861"
+          ixy="-155.063"
+          ixz="40.426"
+          iyy="488.660"
+          iyz="20.213"
+          izz="583.591" />
       </inertial>
       <visual>
@@ -52,4 +52,18 @@
     <link
       name="plate">
+      <inertial>
+        <origin
+          xyz="0 0 0"
+          rpy="0 0 0" />
+        <mass
+          value="0.5" />
+        <inertia
+          ixx="0.007"
+          ixy="0"
+          ixz="0"
+          iyy="0.014"
+          iyz="0"
+          izz="0.007" />
+      </inertial>
       <visual>
         <origin

Commit message: fixed the table angle

File: iiwa_stack/iiwa_description/urdf/rosie2siegmundbase.xacro (robot description, xacro)
@@ -29,5 +29,5 @@
         <origin
           xyz="0 0 0"
-          rpy="0 0 0" />
+          rpy="0 0 1.5708" />
         <geometry>
           <mesh
@@ -43,5 +43,5 @@
         <origin
           xyz="0 0 0"
-          rpy="0 0 0" />
+          rpy="0 0 1.5708" />
         <geometry>
           <mesh
@@ -93,10 +93,12 @@
       <parent link="base"/>
       <child link="plate"/>
-      <origin xyz="0.375 0.475 0.010001" rpy="1.5708 0 0" />
+      <origin xyz="-0.475 0.375 0.010001" rpy="1.5708 0 0" />
     </joint>
+<!--  <origin xyz="0.375 0.475 0.010001" rpy="1.5708 0 0" />
+    </joint>-->
     <joint name="base_adjustment" type="fixed">
       <parent link="plate"/>
       <child link="base_link"/>
-      <origin xyz="0 0.01025 0" rpy="-1.5708 0 0"/>
+      <origin xyz="0 0.01025 0" rpy="-1.5708 1.5708 0"/>
     </joint>
     <link name="base_link"/>
