Commit message: Fixed tcp position

File: src/robotiq/robotiq_2f_85_gripper_visualization/urdf/robotiq_arg2f_85_model_macro.xacro (robot description, xacro)
@@ -9,4 +9,12 @@
       <axis xyz="0 0 0" />
     </joint>
+  <!-- link and joint to updated iiwa TCP (should be moved to separate file) -->
+  <link name="tcp"/>
+  <joint name="tcp_fixed_joint" type="fixed">
+      <origin xyz="0 0 0.130" rpy="0 0 0"/>
+      <parent link="robotiq_arg2f_base_link" />
+      <child link="tcp" />
+      <axis xyz="0 0 0" />
+    </joint>
   <xacro:macro name="outer_knuckle" params="prefix fingerprefix stroke">
     <link name="${prefix}${fingerprefix}_outer_knuckle">
