Commit message: Final Challenge (Ubuntu) commit

File: src/iiwa_stack/iiwa_description/urdf/rosie2siegmundbase.xacro (robot description, xacro)
@@ -29,5 +29,5 @@
         <origin
           xyz="0 0 0"
-          rpy="0 0 0" />
+          rpy="0 0 1.5708" />
         <geometry>
           <mesh
@@ -43,5 +43,5 @@
         <origin
           xyz="0 0 0"
-          rpy="0 0 0" />
+          rpy="0 0 1.5708" />
         <geometry>
           <mesh
@@ -93,10 +93,10 @@
       <parent link="base"/>
       <child link="plate"/>
-      <origin xyz="0.375 0.475 0.010001" rpy="1.5708 0 0" />
+      <origin xyz="-0.475 0.375 0.010001" rpy="1.5708 0 0" />
     </joint>
     <joint name="base_adjustment" type="fixed">
       <parent link="plate"/>
       <child link="base_link"/>
-      <origin xyz="0 0.01025 0" rpy="-1.5708 0 0"/>
+      <origin xyz="0 0.01025 0" rpy="-1.5708 1.5708 0"/>
     </joint>
     <link name="base_link"/>

File: src/robotiq/robotiq_2f_85_gripper_visualization/urdf/robotiq_arg2f_85_model_macro.xacro (robot description, xacro)
@@ -7,5 +7,5 @@
       <parent link="iiwa_link_ee" />
       <child link="robotiq_arg2f_base_link" />
-      <axis xyz="0 0 0" />
+      <!-- <axis xyz="0 0 0" /> -->
     </joint>
   <!-- link and joint to updated iiwa TCP (should be moved to separate file) -->
@@ -15,5 +15,5 @@
       <parent link="robotiq_arg2f_base_link" />
       <child link="tcp" />
-      <axis xyz="0 0 0" />
+      <!-- <axis xyz="0 0 0" /> -->
     </joint>
   <xacro:macro name="outer_knuckle" params="prefix fingerprefix stroke">
